File: LFR_2/LFR_2.kicad_sch (KiCad schematic)
At the start: 10 parts, among them IC1 ESP32-DEVKITC-VE, J1 MOTOR 1, J2 MOTOR 2, J3 BATTERY, SW1 SW_SPST, U1 ROB-14450, U2 TCRT5000L, U3 YAAJ_DCDC_StepDown_LM2596

Commit message: Add files via upload
Parts:
- removed IC1: ESP32-DEVKITC-VE, ESP32DEVKITCVE, symbol ESP32-DEVKITC-VE:ESP32-DEVKITC-VE
- added U15: ESP32-S3-WROOM-1, RF_Module:ESP32-S3-WROOM-1, symbol RF_Module:ESP32-S3-WROOM-1
Connections:
- net +3.3V: no longer U2.1, U2.4
- net AIN 1: now also U15.34 (IO41)
- net AIN 2: now also U15.35 (IO42)
- net BIN 1: now also U15.26 (IO45)
- net BIN 2: now also U15.16 (IO46)
- net ENC_A: now also U15.11 (IO18)
- net ENC_B: now also U15.31 (IO38)
- net ENC_C: now also U15.32 (IO39)
- net ENC_D: now also U15.33 (IO40)
- net GND: now also U15.1 (GND), U15.40 (GND), U15.41 (GND)
- net IR1: now also U15.39 (IO1)
- net IR10: now also U15.18 (IO10)
- net IR11: now also U15.19 (IO11)
- net IR12: now also U15.20 (IO12)
- net IR2: now also U15.38 (IO2)
- net IR3: now also U15.15 (IO3)
- net IR4: now also U15.4 (IO4)
- net IR5: now also U15.5 (IO5)
- net IR6: now also U15.6 (IO6)
- net IR7: now also U15.7 (IO7)
- net IR8: now also U15.12 (IO8)
- net IR9: now also U15.17 (IO9)
- net PWMA A: now also U15.8 (IO15)
- net PWMA B: now also U15.9 (IO16)
- net V BUCK: now also U2.1, U2.4, U15.2 (3V3)
- no-connect marks 0 -> 15
Other:
- moved on the sheet: SW1
